File: hardware/AIC8800M40B/vsf_aic8800m40b.kicad_pcb (KiCad board)
At the start: 4 copper layers, 36.8 x 57.2 mm, 86 parts, among them J1 USB_A, J2 USB_C_Receptacle_USB2.0, J3 USB_C_Receptacle_USB2.0, J4 Micro_SD_Card_Det1, J6 Conn_Coaxial, J7 Conn_Coaxial, J8 Conn_02x15_Odd_Even, Q1 S9013, SW1 SW_Push, SW2 SW_Push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

Commit message: [hardware/aic8800m40b] update
Connections:
- J8 pad 26: /_USB_DM -> unconnected-(J8-Pin_26-Pad26)
- J8 pad 28: /_USB_DP -> unconnected-(J8-Pin_28-Pad28)
Routing:
- net /_USB_DM: track 40.7 -> 18.3 mm, vias 3 -> 2
- net /_USB_DP: track 39.7 -> 18.2 mm, vias 3 -> 2
Other:
- board text added: "3V3 NC"
- board text added: "GND NC"
- board text removed: "3V3 D+"
- board text removed: "GND D-"
Changed lines of the file:
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@@
   (net 83 "unconnected-(J8-Pin_23-Pad23)")
   (net 84 "unconnected-(J8-Pin_24-Pad24)")
+  (net 85 "unconnected-(J8-Pin_26-Pad26)")
+  (net 86 "unconnected-(J8-Pin_28-Pad28)")
   (footprint "Package_TO_SOT_SMD:SOT-23" (layer "F.Cu")
     (at 214.884 119.9665 -90)
@@
       (net 1 "GND") (pinfunction "Pin_25") (pintype "passive"))
     (pad "26" thru_hole oval (at 2.54 30.48) (size 1.7 1.7) (drill 1) (layers "*.Cu" "*.Mask")
-      (net 33 "/_USB_DM") (pinfunction "Pin_26") (pintype "passive"))
+      (net 85 "unconnected-(J8-Pin_26-Pad26)") (pinfunction "Pin_26") (pintype "passive"))
     (pad "27" thru_hole oval (at 0 33.02) (size 1.7 1.7) (drill 1) (layers "*.Cu" "*.Mask")
       (net 5 "/PWR_3V3") (pinfunction "Pin_27") (pintype "passive"))
     (pad "28" thru_hole oval (at 2.54 33.02) (size 1.7 1.7) (drill 1) (layers "*.Cu" "*.Mask")
-      (net 31 "/_USB_DP") (pinfunction "Pin_28") (pintype "passive"))
+      (net 86 "unconnected-(J8-Pin_28-Pad28)") (pinfunction "Pin_28") (pintype "passive"))
     (pad "29" thru_hole oval (at 0 35.56) (size 1.7 1.7) (drill 1) (layers "*.Cu" "*.Mask")
       (net 21 "/USB5V_OUT") (pinfunction "Pin_29") (pintype "passive"))
@@
     (effects (font (size 0.762 0.762) (thickness 0.1524) bold) (justify left bottom))
   )
-  (gr_text "GND\nD-" (at 234.95 137.541 90) (layer "F.SilkS")
+  (gr_text "GND\nNC" (at 234.95 137.541 90) (layer "F.SilkS")
     (effects (font (size 0.635 0.635) (thickness 0.1524) bold) (justify left bottom))
   )
-  (gr_text "3V3\nD+" (at 234.95 140.081 90) (layer "F.SilkS")
+  (gr_text "3V3\nNC" (at 234.95 140.081 90) (layer "F.SilkS")
     (effects (font (size 0.635 0.635) (thickness 0.1524) bold) (justify left bottom))
   )
@@
   (segment (start 209.7909 142.99) (end 211.086 142.99) (width 0.1524) (layer "F.Cu") (net 31))
   (segment (start 209.7909 141.99) (end 211.07 141.99) (width 0.1524) (layer "F.Cu") (net 31))
-  (segment (start 235.7628 137.9728) (end 237.7948 137.9728) (width 0.1524) (layer "F.Cu") (net 31))
-  (segment (start 235.1532 140.7668) (end 235.1532 138.5824) (width 0.1524) (layer "F.Cu") (net 31))
-  (segment (start 222.3008 142.8496) (end 233.0704 142.8496) (width 0.1524) (layer "F.Cu") (net 31))
-  (segment (start 237.7948 137.9728) (end 238.887 139.065) (width 0.1524) (layer "F.Cu") (net 31))
-  (segment (start 235.1532 138.5824) (end 235.7628 137.9728) (width 0.1524) (layer "F.Cu") (net 31))
-  (segment (start 221.9452 143.2052) (end 222.3008 142.8496) (width 0.1524) (layer "F.Cu") (net 31))
   (segment (start 211.086 142.99) (end 211.1756 142.9004) (width 0.1524) (layer "F.Cu") (net 31))
   (segment (start 211.07 141.99) (end 211.1756 141.8844) (width 0.1524) (layer "F.Cu") (net 31))
-  (segment (start 233.0704 142.8496) (end 235.1532 140.7668) (width 0.1524) (layer "F.Cu") (net 31))
   (segment (start 211.582 141.478) (end 211.834 141.478) (width 0.1524) (layer "F.Cu") (net 31))
   (via (at 211.1756 141.8844) (size 0.45212) (drill 0.2032) (layers "F.Cu" "B.Cu") (net 31))
   (via (at 211.1756 142.9004) (size 0.45212) (drill 0.2032) (layers "F.Cu" "B.Cu") (net 31))
-  (via (at 221.9452 143.2052) (size 0.45212) (drill 0.2032) (layers "F.Cu" "B.Cu") (net 31))
-  (segment (start 221.9452 143.2052) (end 222.0188 143.1316) (width 0.1524) (layer "B.Cu") (net 31))
-  (segment (start 222.0188 143.1316) (end 222.615 143.1316) (width 0.1524) (layer "B.Cu") (net 31))
   (segment (start 215.4936 142.9004) (end 217.424 140.97) (width 0.1524) (layer "B.Cu") (net 31))
   (segment (start 217.424 140.97) (end 221.0816 140.97) (width 0.1524) (layer "B.Cu") (net 31))
@@
   (segment (start 210.6676 142.494) (end 210.7692 142.3924) (width 0.1524) (layer "F.Cu") (net 33))
   (segment (start 210.6676 141.478) (end 210.6556 141.49) (width 0.1524) (layer "F.Cu") (net 33))
-  (segment (start 237.7948 137.6172) (end 238.887 136.525) (width 0.1524) (layer "F.Cu") (net 33))
   (segment (start 210.6556 141.49) (end 209.7909 141.49) (width 0.1524) (layer "F.Cu") (net 33))
-  (segment (start 235.6485 137.6172) (end 237.7948 137.6172) (width 0.1524) (layer "F.Cu") (net 33))
   (segment (start 210.6676 141.478) (end 210.7692 141.3764) (width 0.1524) (layer "F.Cu") (net 33))
   (segment (start 211.7324 142.3924) (end 211.834 142.494) (width 0.1524) (layer "F.Cu") (net 33))
   (segment (start 210.7692 142.3924) (end 211.7324 142.3924) (width 0.1524) (layer "F.Cu") (net 33))
-  (segment (start 232.9434 142.494) (end 234.7976 140.6398) (width 0.1524) (layer "F.Cu") (net 33))
   (segment (start 210.6676 142.494) (end 210.6636 142.49) (width 0.1524) (layer "F.Cu") (net 33))
-  (segment (start 234.7976 140.6398) (end 234.7976 138.4681) (width 0.1524) (layer "F.Cu") (net 33))
-  (segment (start 221.2848 143.2052) (end 221.2848 143.1544) (width 0.1524) (layer "F.Cu") (net 33))
-  (segment (start 221.9452 142.494) (end 232.9434 142.494) (width 0.1524) (layer "F.Cu") (net 33))
-  (segment (start 221.2848 143.1544) (end 221.9452 142.494) (width 0.1524) (layer "F.Cu") (net 33))
-  (segment (start 234.7976 138.4681) (end 235.6485 137.6172) (width 0.1524) (layer "F.Cu") (net 33))
   (segment (start 210.6636 142.49) (end 209.7909 142.49) (width 0.1524) (layer "F.Cu") (net 33))
   (via (at 210.6676 141.478) (size 0.45212) (drill 0.2032) (layers "F.Cu" "B.Cu") (net 33))
-  (via (at 221.2848 143.2052) (size 0.45212) (drill 0.2032) (layers "F.Cu" "B.Cu") (net 33))
   (via (at 210.6676 142.494) (size 0.45212) (drill 0.2032) (layers "F.Cu" "B.Cu") (net 33))
   (segment (start 221.3356 142.411) (end 220.615 143.1316) (width 0.1524) (layer "B.Cu") (net 33))
   (segment (start 215.4936 143.4084) (end 217.551 141.351) (width 0.1524) (layer "B.Cu") (net 33))
   (segment (start 210.6676 142.494) (end 210.6676 143.1544) (width 0.1524) (layer "B.Cu") (net 33))
-  (segment (start 221.2848 143.2052) (end 221.2112 143.1316) (width 0.1524) (layer "B.Cu") (net 33))
-  (segment (start 221.2112 143.1316) (end 220.615 143.1316) (width 0.1524) (layer "B.Cu") (net 33))
   (segment (start 220.9546 141.351) (end 221.3356 141.732) (width 0.1524) (layer "B.Cu") (net 33))
   (segment (start 210.6676 141.478) (end 210.6676 142.494) (width 0.1524) (layer "B.Cu") (net 33))
