File: hardware/AIC8800M40B/vsf_aic8800m40b.kicad_sch (KiCad schematic)
At the start: 86 parts, among them J1 USB_A, J2 USB_C_Receptacle_USB2.0, J3 USB_C_Receptacle_USB2.0, J4 Micro_SD_Card_Det1, J6 Conn_Coaxial, J7 Conn_Coaxial, J8 Conn_02x15_Odd_Even, Q1 S9013, SW1 SW_Push, SW2 SW_Push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

Commit message: [hardware/aic8800m40b] update
Connections:
- net _USB_DM: no longer J8.26 (Pin_26)
- net _USB_DP: no longer J8.28 (Pin_28)
Changed lines of the file:
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@@
-    (effects (font (size 1.27 1.27)) (justify left bottom))
-  )
-  (label "_USB_DP" (at 39.37 55.88 0) (fields_autoplaced)
     (effects (font (size 1.27 1.27)) (justify left bottom))
   )
@@
     (effects (font (size 1.27 1.27)) (justify left bottom))
   )
-  (label "_USB_DM" (at 39.37 53.34 0) (fields_autoplaced)
-    (effects (font (size 1.27 1.27)) (justify left bottom))
-  )
